File: eagle/xsa2-servo-pcb/servo-pcb.brd (EAGLE design)
At the start: 160 x 100 mm, 44 parts, among them IC1 ESP32-WROOM-32D__4MB_PS_, IC2 FT231XS-R, IC3 NJM2884U1-33-TE1, IC4 TPA2006D1DRBR, IC5 ISL90728UIE627Z-TK, J1 WJEK254-2.54-02P-140-00A, J2 CX70M-24P1, J3 WJEK254-2.54-02P-140-00A, J4 WJEK254-2.54-02P-140-00A, Q1 IRLML6402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

Commit message: [eagle] 回路追加
Connections:
- removed net N$35: IC2.1, JP5.6
- new net DTR: IC2.1, S2.5
- new net N$17: JP5.6, S2.4
- new net N$41: JP5.5, S2.1
- new net RXD: IC2.4, S2.2
- net N$11: now also S2.6; no longer IC2.9
- net N$16: now also S2.3; no longer IC2.4, JP5.5
Changed lines of the file:
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@@
 <contactref element="R8" pad="1"/>
 <contactref element="Q2" pad="2"/>
-<contactref element="IC2" pad="9"/>
-<wire x1="-52.92" y1="62.23" x2="-19.67" y2="66.36" width="0" layer="19" extent="1-1"/>
-<wire x1="-34.462" y1="32.068" x2="-52.92" y2="62.23" width="0" layer="19" extent="1-1"/>
+<contactref element="S2" pad="6"/>
+<wire x1="-52.92" y1="62.23" x2="-110.53" y2="-23.24" width="0" layer="19" extent="1-1"/>
+<wire x1="-19.67" y1="66.36" x2="-52.92" y2="62.23" width="0" layer="19" extent="1-1"/>
 </signal>
 <signal name="N$12">
@@
 </signal>
 <signal name="N$16">
-<contactref element="IC2" pad="4"/>
 <contactref element="IC1" pad="35"/>
-<contactref element="JP5" pad="5"/>
-<wire x1="-34.462" y1="35.242" x2="-111.76" y2="-6.35" width="0" layer="19" extent="1-1"/>
-<wire x1="-19.44" y1="16.69" x2="-34.462" y2="35.242" width="0" layer="19" extent="1-1"/>
-</signal>
-<signal name="N$17">
-<contactref element="IC2" pad="20"/>
-<contactref element="IC1" pad="34"/>
-<contactref element="JP5" pad="4"/>
-<wire x1="-29.038" y1="37.148" x2="-114.3" y2="-3.81" width="0" layer="19" extent="1-1"/>
-<wire x1="-19.44" y1="15.42" x2="-29.038" y2="37.148" width="0" layer="19" extent="1-1"/>
+<contactref element="S2" pad="3"/>
+<wire x1="-19.44" y1="16.69" x2="-110.53" y2="-19.94" width="0" layer="19" extent="1-1"/>
 </signal>
 <signal name="N$18">
@@
 </signal>
 <signal name="VDD">
-<contactref element="Q1" pad="3"/>
-<contactref element="R2" pad="1"/>
-<contactref element="C1" pad="1"/>
-<contactref element="IC3" pad="6"/>
 <contactref element="IC4" pad="6"/>
 <contactref element="J3" pad="2"/>
@@
 <contactref element="JP2" pad="2"/>
 <contactref element="JP5" pad="12"/>
+<contactref element="Q1" pad="3"/>
+<contactref element="R2" pad="1"/>
+<contactref element="C1" pad="1"/>
+<contactref element="IC3" pad="6"/>
 <wire x1="-104.14" y1="-3.81" x2="-113.03" y2="2.54" width="0" layer="19" extent="1-1"/>
 <wire x1="-100.33" y1="2.54" x2="-104.14" y2="-3.81" width="0" layer="19" extent="1-1"/>
@@
 <wire x1="-36.44" y1="10.34" x2="-115.57" y2="2.54" width="0" layer="19" extent="1-1"/>
 </signal>
-<signal name="N$35">
-<contactref element="IC2" pad="1"/>
-<contactref element="JP5" pad="6"/>
-<wire x1="-34.462" y1="37.148" x2="-111.76" y2="-3.81" width="0" layer="19" extent="1-1"/>
-</signal>
 <signal name="N$34">
 <contactref element="IC1" pad="27"/>
@@
 <wire x1="-19.44" y1="9.07" x2="-104.14" y2="-6.35" width="0" layer="19" extent="1-1"/>
 </signal>
+<signal name="N$40">
+<contactref element="IC1" pad="34"/>
+<contactref element="IC2" pad="20"/>
+<contactref element="JP5" pad="4"/>
+<wire x1="-29.038" y1="37.148" x2="-114.3" y2="-3.81" width="0" layer="19" extent="1-1"/>
+<wire x1="-19.44" y1="15.42" x2="-29.038" y2="37.148" width="0" layer="19" extent="1-1"/>
+</signal>
+<signal name="RXD">
+<contactref element="IC2" pad="4"/>
+<contactref element="S2" pad="2"/>
+<wire x1="-34.462" y1="35.242" x2="-113.03" y2="-19.94" width="0" layer="19" extent="1-1"/>
+</signal>
+<signal name="DTR">
+<contactref element="IC2" pad="1"/>
+<contactref element="S2" pad="5"/>
+<wire x1="-34.462" y1="37.148" x2="-113.03" y2="-23.24" width="0" layer="19" extent="1-1"/>
+</signal>
+<signal name="N$17">
+<contactref element="S2" pad="4"/>
+<contactref element="JP5" pad="6"/>
+<wire x1="-111.76" y1="-3.81" x2="-115.53" y2="-23.24" width="0" layer="19" extent="1-1"/>
+</signal>
+<signal name="N$41">
+<contactref element="S2" pad="1"/>
+<contactref element="JP5" pad="5"/>
+<wire x1="-111.76" y1="-6.35" x2="-115.53" y2="-19.94" width="0" layer="19" extent="1-1"/>
+</signal>
 </signals>

Commit message: [eagle] 回路図更新
Parts:
- removed J2: CX70M-24P1, CX70M-24P1:HRS_CX70M-24P1
- added U$1: 5077CR-16-SMC2-BK-TR, FaBo-Connetor:5077CR-16SMC2-BK-TR
Connections:
- removed net N$4: J2.B5, R4.2
- removed net N$6: J2.A5, R3.2
- new net N$35: R4.2, U$1.B5:CC2
- new net N$42: R3.2, U$1.A5:CC1
- net GND: now also U$1.A1,B12:GND, U$1.B1,A12:GND; no longer J2.A1, J2.A12, J2.B1, J2.B12, J2.S1, J2.S2, J2.S3, J2.S4, J2.S5, J2.S5.1, J2.S6, J2.S6.1
- net N$1: now also U$1.A6:DP1, U$1.B6:DP2; no longer J2.A6, J2.B6
- net N$5: now also U$1.A7:DN1, U$1.B7:DN2; no longer J2.A7, J2.B7
- net VCC: now also U$1.A4,B9:V_BUS; no longer J2.A4, J2.A9, J2.B4, J2.B9
