File: eagle/xsa2-servo-pcb/servo-pcb-sheet.brd (EAGLE design)
At the start: 96 x 85 mm, 45 parts, among them IC1 ESP32-WROOM-32D__4MB_PS_, IC2 FT231XS-R, IC3 NJM2884U1-33-TE1, IC4 TPA2006D1DRBR, IC5 ISL90728UIE627Z-TK, J1 WJEK254-2.54-02P-140-00A, J3 WJEK254-2.54-02P-140-00A, J4 WJEK254-2.54-02P-140-00A, Q1 IRLML6402, Q2 2SC2712-GR_F_, Q3 2SC2712-GR_F_

Commit message: [eagle] サーボ基板完成
Parts:
- moved FL1 1.81 mm to (35.4, 27.6), flipped to the bottom, turned to 0 degrees
Routing:
- net VDD: track 50.4 -> 48.6 mm, vias 3 -> 2
- net N$38: track 10.3 -> 12.0 mm, vias 0 -> 1
- net N$13: track 22.2 -> 22.8 mm
- net GND: vias 40 -> 45
Other:
- board text added: "XSA Servo PCB V1.0 ailab*"

Commit message: [eagle] サーボ基板の面付け
Parts:
- added C10, C19, C28: 0.33uF, rcl:C0603
- added C11, C15, C16, C20, C24, C25, C29, C33, C34: 1uF, rcl:C0603
- added C12, C13, C21, C22, C30, C31: 39pF, rcl:C0603
- added C14, C17, C23, C26, C32, C35: 10uF, rcl:C0805
- added C18, C27, C36: 0.01uF, rcl:C0603
- added FL2, FL3, FL4: BLM18PG121SN1D, SamacSys_Parts:BLM18AG102BH1D
- added IC10, IC15, IC20: ISL90728UIE627Z-TK, SamacSys_Parts:SOT65P210X110-6N
- added IC11, IC16, IC6: ESP32-WROOM-32D__4MB_PS_, SamacSys_Parts:ESP32WROOM32D4MBPS
- added IC12, IC17, IC7: FT231XS-R, SamacSys_Parts:SOP64P599X175-20N
- added IC13, IC18, IC8: NJM2884U1-33-TE1, SamacSys_Parts:SOT-89-5-1
- added IC14, IC19, IC9: TPA2006D1DRBR, SamacSys_Parts:TPA2006D1DRBR
- added J10, J11, J12, J2, J5, J6, J7, J8, J9: WJEK254-2.54-02P-140-00A, SamacSys_Parts:WJEK25425402P14000A
- added JP10, JP3, JP7: SERVO1, pinhead:2X03/90
- added JP11, JP4, JP8: SERVO2, pinhead:2X03/90
- added JP12, JP6, JP9: (no value), pinhead:2X07
- added Q10, Q4, Q7: IRLML6402, SamacSys_Parts:SOT95P237X112-3N
- added Q11, Q12, Q5, Q6, Q8, Q9: 2SC2712-GR_F_, SamacSys_Parts:SSM3K7002CFULF
- added R19, R20, R21, R22, R37, R38, R39, R40, R55, R56, R57, R58: 10k, rcl:R0603
- added R23, R24, R41, R42, R59, R60: 100k, rcl:R0603
- added R25, R33, R34, R43, R51, R52, R61, R69, R70: 1k, rcl:R0603
- added R26, R27, R32, R44, R45, R50, R62, R63, R68: 4.7k, rcl:R0603
- added R28, R29, R46, R47, R64, R65: 27, rcl:R0603
- added R30, R31, R48, R49, R66, R67: 12k, rcl:R0603
- added R35, R36, R53, R54, R71, R72: 0, rcl:R0603
- added S3, S5, S7: SK-12D11VG3, SamacSys_Parts:SK12D11VG3
- added S4, S6, S8: IS-2235, SamacSys_Parts:IS2235
- added U$2, U$3, U$4: 5077CR-16-SMC2-BK-TR, FaBo-Connetor:5077CR-16SMC2-BK-TR
Connections:
- new net +3V1: C11.1, C14.1, C17.1, C18.1, IC10.1, IC6.2, IC7.13, IC7.14, IC7.15, IC7.3, IC8.4, JP6.8, R21.2, R22.2, R33.2, R34.2
- new net +3V2: C20.1, C23.1, C26.1, C27.1, IC11.2, IC12.13, IC12.14, IC12.15, IC12.3, IC13.4, IC15.1, JP9.8, R39.2, R40.2, R51.2, R52.2
- new net +3V4: C29.1, C32.1, C35.1, C36.1, IC16.2, IC17.13, IC17.14, IC17.15, IC17.3, IC18.4, IC20.1, JP12.8, R57.2, R58.2, R69.2, R70.2
- new net DTR1: IC7.1, S4.5
- new net DTR2: IC12.1, S6.5
- new net DTR3: IC17.1, S8.5
- new net GND1: C10.2, C11.2, C12.2, C13.2, C14.2, C16.2, C17.2, C18.2, IC10.2, IC6.1, IC6.15, IC6.38, IC6.39, IC6.40, IC6.41, IC6.42, IC6.43, IC6.44, IC6.45, IC6.46, IC6.47, IC7.16, IC7.6, IC8.2, IC8.5, IC9.7, J6.2, JP3.5, JP3.6, JP4.5, JP4.6, JP6.1, JP6.2, R20.1, R26.1, R27.1, S3.2, S3.MH1, S3.MH2, U$2.A1,B12:GND, U$2.B1,A12:GND
- new net GND2: C19.2, C20.2, C21.2, C22.2, C23.2, C25.2, C26.2, C27.2, IC11.1, IC11.15, IC11.38, IC11.39, IC11.40, IC11.41, IC11.42, IC11.43, IC11.44, IC11.45, IC11.46, IC11.47, IC12.16, IC12.6, IC13.2, IC13.5, IC14.7, IC15.2, J9.2, JP7.5, JP7.6, JP8.5, JP8.6, JP9.1, JP9.2, R38.1, R44.1, R45.1, S5.2, S5.MH1, S5.MH2, U$3.A1,B12:GND, U$3.B1,A12:GND
- new net GND3: C28.2, C29.2, C30.2, C31.2, C32.2, C34.2, C35.2, C36.2, IC16.1, IC16.15, IC16.38, IC16.39, IC16.40, IC16.41, IC16.42, IC16.43, IC16.44, IC16.45, IC16.46, IC16.47, IC17.16, IC17.6, IC18.2, IC18.5, IC19.7, IC20.2, J12.2, JP10.5, JP10.6, JP11.5, JP11.6, JP12.1, JP12.2, R56.1, R62.1, R63.1, S7.2, S7.MH1, S7.MH2, U$4.A1,B12:GND, U$4.B1,A12:GND
- new net IO1: IC6.14, JP6.9
- new net IO2: JP6.10, R35.2, R36.2
- new net IO3: IC11.14, JP9.9
- new net IO4: JP9.10, R53.2, R54.2
- new net IO5: IC16.14, JP12.9
- new net IO6: JP12.10, R71.2, R72.2
- new net N$100: IC11.13, IC14.1
- new net N$101: IC14.8, J7.1
- new net N$102: IC14.5, J7.2
- new net N$103: IC11.10, IC15.6
- new net N$104: IC11.11, JP7.1
- new net N$105: IC11.12, JP7.2
- new net N$106: IC11.8, JP8.1
- new net N$107: IC11.9, JP8.2
- new net N$108: IC11.27, JP9.13
- new net N$109: JP9.7, S6.4
- new net N$110: JP9.6, S6.1
- new net N$111: R45.2, U$3.B5:CC2
- new net N$112: R44.2, U$3.A5:CC1
- new net N$113: IC11.28, JP9.14
- new net N$114: IC11.34, IC12.20, JP9.5
- new net N$115: IC11.16, J8.1, R53.1
- new net N$116: J9.1, R54.1
- new net N$117: FL3.1, JP7.3, JP7.4, JP8.3, JP8.4
- new net N$118: Q10.1, R55.1, S7.1
- new net N$119: IC18.1, R61.2
- new net N$120: C31.1, R65.1, U$4.A6:DP1, U$4.B6:DP2
- new net N$121: C30.1, R64.1, U$4.A7:DN1, U$4.B7:DN2
- new net N$122: IC17.12, R64.2
- new net N$123: IC17.11, R65.2
- new net N$124: IC17.2, Q12.3, R66.1
- new net N$125: Q11.1, R66.2
- new net N$126: Q11.2, R67.1, S8.6
- new net N$127: Q12.1, R67.2
- new net N$128: IC17.18, R56.2, R68.1
- new net N$129: IC16.3, Q12.2, R58.1
- new net N$130: IC16.25, Q11.3, R57.1
- new net N$131: IC16.35, S8.3
- new net N$132: IC20.5, R59.1
- new net N$133: C33.1, R59.2
- new net N$134: C33.2, IC19.4
- new net N$135: IC19.3, R60.2
- new net N$136: C34.1, R60.1
- new net N$137: IC16.36, IC20.3, JP12.4, R69.1
- new net N$138: IC16.33, IC20.4, JP12.3, R70.1
- new net N$139: IC16.13, IC19.1
- new net N$140: IC19.8, J10.1
- new net N$141: IC19.5, J10.2
- new net N$142: IC16.10, IC20.6
- new net N$143: IC16.11, JP10.1
- new net N$144: IC16.12, JP10.2
- new net N$145: IC16.8, JP11.1
- new net N$146: IC16.9, JP11.2
- new net N$147: IC16.27, JP12.13
- new net N$148: JP12.7, S8.4
- new net N$149: JP12.6, S8.1
- new net N$150: R63.2, U$4.B5:CC2
- new net N$151: R62.2, U$4.A5:CC1
- new net N$152: IC16.28, JP12.14
- new net N$153: IC16.34, IC17.20, JP12.5
- new net N$154: IC16.16, J11.1, R71.1
- new net N$155: J12.1, R72.1
- new net N$156: FL4.1, JP10.3, JP10.4, JP11.3, JP11.4
- new net N$37: Q4.1, R19.1, S3.1
- new net N$39: IC8.1, R25.2
- new net N$40: C13.1, R29.1, U$2.A6:DP1, U$2.B6:DP2
- new net N$43: C12.1, R28.1, U$2.A7:DN1, U$2.B7:DN2
- new net N$44: IC7.12, R28.2
- new net N$45: IC7.11, R29.2
- new net N$46: IC7.2, Q6.3, R30.1
- new net N$47: Q5.1, R30.2
- new net N$48: Q5.2, R31.1, S4.6
- new net N$49: Q6.1, R31.2
- new net N$50: IC7.18, R20.2, R32.1
- new net N$51: IC6.3, Q6.2, R22.1
- new net N$52: IC6.25, Q5.3, R21.1
- new net N$53: IC6.35, S4.3
- new net N$54: IC10.5, R23.1
- new net N$55: C15.1, R23.2
- new net N$56: C15.2, IC9.4
- new net N$57: IC9.3, R24.2
- new net N$58: C16.1, R24.1
- new net N$59: IC10.3, IC6.36, JP6.4, R33.1
- new net N$60: IC10.4, IC6.33, JP6.3, R34.1
- new net N$61: IC6.13, IC9.1
- new net N$62: IC9.8, J2.1
- new net N$63: IC9.5, J2.2
- new net N$64: IC10.6, IC6.10
- new net N$65: IC6.11, JP3.1
- new net N$66: IC6.12, JP3.2
- new net N$67: IC6.8, JP4.1
- new net N$68: IC6.9, JP4.2
- new net N$69: IC6.27, JP6.13
- new net N$70: JP6.7, S4.4
- new net N$71: JP6.6, S4.1
- new net N$72: R27.2, U$2.B5:CC2
- new net N$73: R26.2, U$2.A5:CC1
- new net N$74: IC6.28, JP6.14
- new net N$75: IC6.34, IC7.20, JP6.5
- new net N$76: IC6.16, J5.1, R35.1
- new net N$77: J6.1, R36.1
- new net N$78: FL2.1, JP3.3, JP3.4, JP4.3, JP4.4
- new net N$79: Q7.1, R37.1, S5.1
- new net N$80: IC13.1, R43.2
- new net N$81: C22.1, R47.1, U$3.A6:DP1, U$3.B6:DP2
- new net N$82: C21.1, R46.1, U$3.A7:DN1, U$3.B7:DN2
- new net N$83: IC12.12, R46.2
- new net N$84: IC12.11, R47.2
- new net N$85: IC12.2, Q9.3, R48.1
- new net N$86: Q8.1, R48.2
- new net N$87: Q8.2, R49.1, S6.6
- new net N$88: Q9.1, R49.2
- new net N$89: IC12.18, R38.2, R50.1
- new net N$90: IC11.3, Q9.2, R40.1
- new net N$91: IC11.25, Q8.3, R39.1
- new net N$92: IC11.35, S6.3
- new net N$93: IC15.5, R41.1
- new net N$94: C24.1, R41.2
- new net N$95: C24.2, IC14.4
- new net N$96: IC14.3, R42.2
- new net N$97: C25.1, R42.1
- new net N$98: IC11.36, IC15.3, JP9.4, R51.1
- new net N$99: IC11.33, IC15.4, JP9.3, R52.1
- new net RXD1: IC7.4, S4.2
- new net RXD2: IC12.4, S6.2
- new net RXD3: IC17.4, S8.2
- new net VCC1: Q4.2, R19.2, R32.2, U$2.A4,B9:V_BUS, U$2.B4,A9:VBUS
- new net VCC2: Q7.2, R37.2, R50.2, U$3.A4,B9:V_BUS, U$3.B4,A9:VBUS
- new net VCC3: Q10.2, R55.2, R68.2, U$4.A4,B9:V_BUS, U$4.B4,A9:VBUS
- new net VDD1: C10.1, FL2.2, IC8.6, IC9.6, J5.2, JP6.11, JP6.12, Q4.3, R25.1
- new net VDD2: C19.1, FL3.2, IC13.6, IC14.6, J8.2, JP9.11, JP9.12, Q7.3, R43.1
- new net VDD3: C28.1, FL4.2, IC18.6, IC19.6, J11.2, JP12.11, JP12.12, Q10.3, R61.1
Routing:
- net +3V2: track 0.00 -> 75.4 mm, vias 0 -> 5
- net +3V4: track 0.00 -> 75.4 mm, vias 0 -> 5
- net +3V1: track 0.00 -> 75.4 mm, vias 0 -> 5
- net N$98: track 0.00 -> 68.1 mm, vias 0 -> 1
- net N$59: track 0.00 -> 68.1 mm, vias 0 -> 1
- net N$137: track 0.00 -> 68.1 mm, vias 0 -> 1
- net N$87: track 0.00 -> 62.5 mm, vias 0 -> 2
- net N$48: track 0.00 -> 62.5 mm, vias 0 -> 2
- net N$126: track 0.00 -> 62.5 mm, vias 0 -> 2
- net RXD3: track 0.00 -> 59.5 mm, vias 0 -> 2
- net RXD1: track 0.00 -> 59.5 mm, vias 0 -> 2
- net RXD2: track 0.00 -> 59.5 mm, vias 0 -> 2
- net N$61: track 0.00 -> 53.2 mm, vias 0 -> 1
- net N$139: track 0.00 -> 53.2 mm, vias 0 -> 1
- net N$100: track 0.00 -> 53.2 mm, vias 0 -> 1
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- added copper zone on layer 1, net GND1
- added copper zone on layer 16, net GND1
- added copper zone on layer 1, net GND2
- added copper zone on layer 16, net GND2
- added copper zone on layer 1, net GND3
- added copper zone on layer 16, net GND3
Other:
- board text added: "C1"
- board text added: "C2"
- board text added: "C3"
- board text added: "C4"
- board text added: "C5"
- board text added: "C6"
- board text added: "C7"
- board text added: "C8"
- board text added: "C9"
- board text added: "FL1"
- board text added: "IC1"
- board text added: "IC2"
- board text added: "IC3"
- board text added: "IC4"
- board text added: "IC5"
- board text added: "J1"
- board text added: "J3"
- board text added: "J4"
- board text added: "JP1"
- board text added: "JP2"
- board text added: "JP5"
- board text added: "Q1"
- board text added: "Q2"
- board text added: "Q3"
- board text added: "R1"
- board text added: "R10"
- board text added: "R11"
- board text added: "R12"
- board text added: "R13"
- board text added: "R14"
- board text added: "R15"
- board text added: "R16"
- board text added: "R17"
- board text added: "R18"
- board text added: "R2"
- board text added: "R3"
- board text added: "R4"
- board text added: "R5"
- board text added: "R6"
- board text added: "R7"
- board text added: "R8"
- board text added: "R9"
- board text added: "S1"
- board text added: "S2"
